File: shinobi.brd (EAGLE design)
At the start: 57 x 47 mm, 112 parts, among them J1 2171790001, J2 61300711121, J3 61301011121, J4 61300211121, J5 61300211121, U1 TV5725, U2 W9864G2JH-6, U3 ESP-06, U4 74ABT125PW, U5 Si5351A-B-GT, U6 CH340C, U7 TPS621351, U8 NCV8187AMN180TAG, Y1 27MHZ 10pF, Y2 25.0MHz 10pF

Commit message: update images, add eagle palette script
Parts:
- L2, L3, L4: value ? -> 10uH
- renumbered FB1 to L2, FB2 to L3, FB3 to L4
Changed lines of the file:
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@@
 </element>
 <element name="Y2" library="microbuilder" package="CRYSTAL_2.5X2" value="25.0MHz 10pF" x="15.113" y="6.096" smashed="yes" rot="R90"/>
-<element name="FB1" library="resistor" library_urn="urn:adsk.eagle:library:2745533" package="R0402" package3d_urn="urn:adsk.eagle:package:2745538/3" value="?" x="29.083" y="40.767" smashed="yes"/>
-<element name="FB2" library="resistor" library_urn="urn:adsk.eagle:library:2745533" package="R0402" package3d_urn="urn:adsk.eagle:package:2745538/3" value="?" x="32.893" y="40.767" smashed="yes"/>
-<element name="FB3" library="resistor" library_urn="urn:adsk.eagle:library:2745533" package="R0402" package3d_urn="urn:adsk.eagle:package:2745538/3" value="?" x="38.862" y="40.767" smashed="yes"/>
+<element name="L2" library="resistor" library_urn="urn:adsk.eagle:library:2745533" package="R0402" package3d_urn="urn:adsk.eagle:package:2745538/3" value="10uH" x="29.083" y="40.767" smashed="yes"/>
+<element name="L3" library="resistor" library_urn="urn:adsk.eagle:library:2745533" package="R0402" package3d_urn="urn:adsk.eagle:package:2745538/3" value="10uH" x="32.893" y="40.767" smashed="yes"/>
+<element name="L4" library="resistor" library_urn="urn:adsk.eagle:library:2745533" package="R0402" package3d_urn="urn:adsk.eagle:package:2745538/3" value="10uH" x="38.862" y="40.767" smashed="yes"/>
 <element name="C56" library="resistor" library_urn="urn:adsk.eagle:library:2745533" package="C0402" package3d_urn="urn:adsk.eagle:package:2745540/2" value="15pF" x="29.083" y="41.656" smashed="yes"/>
 <element name="C57" library="resistor" library_urn="urn:adsk.eagle:library:2745533" package="C0402" package3d_urn="urn:adsk.eagle:package:2745540/2" value="15pF" x="32.893" y="41.656" smashed="yes"/>
@@
 <contactref element="J3" pad="1"/>
 <contactref element="C56" pad="2"/>
-<contactref element="FB1" pad="2"/>
+<contactref element="L2" pad="2"/>
 <contactref element="C59" pad="1"/>
 <wire x1="30.5308" y1="41.6988" x2="30.488" y2="41.656" width="0.3048" layer="1"/>
@@
 <contactref element="J3" pad="3"/>
 <contactref element="C57" pad="2"/>
-<contactref element="FB2" pad="2"/>
+<contactref element="L3" pad="2"/>
 <contactref element="C60" pad="1"/>
 <wire x1="33.393" y1="40.767" x2="33.393" y2="41.656" width="0.3048" layer="1"/>
@@
 <contactref element="J3" pad="5"/>
 <contactref element="C58" pad="2"/>
-<contactref element="FB3" pad="2"/>
+<contactref element="L4" pad="2"/>
 <contactref element="C61" pad="1"/>
 <wire x1="39.362" y1="41.656" x2="39.362" y2="40.767" width="0.3048" layer="1"/>
@@
 <contactref element="U1" pad="158"/>
 <contactref element="C58" pad="1"/>
-<contactref element="FB3" pad="1"/>
+<contactref element="L4" pad="1"/>
 <contactref element="R16" pad="1"/>
 <via x="38.354" y="39.878" extent="1-16" drill="0.254" diameter="0.508"/>
@@
 <contactref element="U1" pad="159"/>
 <contactref element="C57" pad="1"/>
-<contactref element="FB2" pad="1"/>
+<contactref element="L3" pad="1"/>
 <contactref element="R17" pad="1"/>
 <via x="32.2326" y="39.878" extent="1-16" drill="0.254" diameter="0.508"/>
@@
 <contactref element="U1" pad="160"/>
 <contactref element="C56" pad="1"/>
-<contactref element="FB1" pad="1"/>
+<contactref element="L2" pad="1"/>
 <contactref element="R18" pad="1"/>
 <via x="27.94" y="40.4876" extent="1-16" drill="0.254" diameter="0.508"/>
