File: KiCAD/shinobi.kicad_pcb (KiCad board)
At the start: 4 copper layers, 49.9 x 47 mm, 111 parts, among them IC1 TPS62825DMQT, IC2 TPS62825DMQT, IC3 74LVC2G17GW-Q100H, J2 61300711121, J3 61301011121, J4 61300211121, J5 USB_C_Receptacle_USB2.0_16P, Q1 UMH3N, U1 TV5725, U2 W9864G2JH-6, U5 SI5351A, U6 CH343P, U7 ESP8285, Y1 CRYSTAL2.5X2.0, Y2 CRYSTAL2.5X2.0, Y3 26MHz

Commit message: shinobi2 routing
Parts:
- removed C29: C-USC0402, Capacitor_SMD:C_0402_1005Metric
- added C66: C_Feedthrough, SamacSys_Parts:NFM18PC106D0J3L, F.Cu at (145.8, 89.5)
- Y1, Y2, Y3: footprint Crystal:Crystal_SMD_2520-4Pin_2.5x2.0mm -> SamacSys_Parts:Crystal_SMD_2520-4Pin_2.5x2.0mm
- moved R20 1.11 mm to (127.2, 96.5)
- moved R21 1.09 mm to (128.3, 96.5)
- moved C12 0.96 mm to (134.1, 98.5), turned to 135 degrees
- moved Y2 0.42 mm to (134.8, 122.0), turned to 90 degrees
- moved C62 0.34 mm to (145.2, 86.6)
- moved R14 0.34 mm to (145.2, 87.6)
- moved C53 0.29 mm to (133.4, 85.6), turned to 110 degrees
- moved C3 0.23 mm to (154.5, 125.0)
- moved R3 0.23 mm to (154.5, 126.8)
- moved C13 0.22 mm to (138.4, 89.5)
- moved C33 0.10 mm to (139.9, 91.7)
Connections:
- net /MBA renamed MBA
- C3 pad 1: unconnected-(C3-Pad1) -> Net-(C3-Pad1)
- C4 pad 1: unconnected-(C4-Pad1) -> Net-(C4-Pad1)
- C5 pad 1: unconnected-(C5-Pad1) -> Net-(C5-Pad1)
- R1 pad 1: unconnected-(R1-Pad1) -> +2V5
- R1 pad 2: unconnected-(R1-Pad2) -> Net-(U1-RSTN)
- R2 pad 2: Net-(U1-DAVS) -> GND
- R3 pad 1: unconnected-(R3-Pad1) -> /R
- R3 pad 2: unconnected-(R3-Pad2) -> Net-(C3-Pad1)
- R4 pad 1: unconnected-(R4-Pad1) -> GND
- R4 pad 2: unconnected-(R4-Pad2) -> /R
- R5 pad 1: unconnected-(R5-Pad1) -> /G
- R5 pad 2: unconnected-(R5-Pad2) -> Net-(C4-Pad1)
- R6 pad 1: unconnected-(R6-Pad1) -> GND
- R6 pad 2: unconnected-(R6-Pad2) -> /G
- R7 pad 1: unconnected-(R7-Pad1) -> /B
- R7 pad 2: unconnected-(R7-Pad2) -> Net-(C5-Pad1)
- R8 pad 1: unconnected-(R8-Pad1) -> GND
- R8 pad 2: unconnected-(R8-Pad2) -> /B
- RN2 pad 5: RST -> SCL
- RN2 pad 6: GPIO2 -> SDA
- RN2 pad 8: CHIP_EN -> GPIO2
- RN3 pad 3: unconnected-(RN3-R3.1-Pad3) -> RST
- RN3 pad 4: unconnected-(RN3-R4.1-Pad4) -> CHIP_EN
- RN3 pad 5: unconnected-(RN3-R4.2-Pad5) -> +2V5
- RN3 pad 6: unconnected-(RN3-R3.2-Pad6) -> +2V5
- U1 pad 122: Net-(U1-DAVS) -> GND
- U1 pad 126: Net-(U1-DAVS) -> GND
- U1 pad 136: Net-(U1-DAVS) -> GND
- U1 pad 143: Net-(U1-DAVS) -> GND
- U1 pad 148: Net-(U1-DAVS) -> GND
- U1 pad 153: Net-(U1-DAVS) -> GND
- U1 pad 156: Net-(U1-DAVS) -> GND
- U1 pad 157: +2V5 -> Net-(U1-DAVD)
- U1 pad 75: unconnected-(U1-RSTN-Pad75) -> Net-(U1-RSTN)
Routing:
- net V: track 0.00 -> 24.7 mm, vias 0 -> 1
- net +1V5: track 13.8 -> 36.6 mm
- net SCL: track 35.3 -> 56.5 mm
- net /DEBUG: track 2.02 -> 23.0 mm, vias 1 -> 2
- net Net-(Q1A-E1): track 0.00 -> 18.7 mm, vias 0 -> 2
- net H: track 0.00 -> 18.2 mm, vias 0 -> 1
- net RST: track 0.64 -> 18.1 mm, vias 1 -> 3
- net SDA: track 36.8 -> 52.6 mm
- net BOUT: track 3.02 -> 18.3 mm, vias 1 -> 2
- net Net-(Q1A-B1): track 0.00 -> 15.3 mm, vias 0 -> 2
- net VBUS: track 0.00 -> 14.4 mm, vias 0 -> 16
- net GOUT: track 3.02 -> 16.5 mm, vias 1 -> 2
- net +2V5: track 84.9 -> 97.4 mm, vias 30 -> 43
- net Net-(J5-CC2): track 0.00 -> 11.4 mm
- net GPIO0: track 0.60 -> 10.9 mm, vias 1 -> 2
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- added copper zone on In2.Cu, net +1V5
- added copper zone on F.Cu, net VBUS

Commit message: Update PCB and BOM
Parts:
- removed the J2 at (136.1, 126.7)
- added J4: 61300711121, shinobi:61300711121_11687645, F.Cu at (136.1, 126.7)
- AE1: value Antenna -> AMCA72-2R470G-S1F-T4
- C18: renamed from C63; value 0.1μF -> 130pF
- C19: renamed from C62; value 0.1μF -> 130pF
- C20: renamed from C17; value C_Feedthrough -> NFM18PC106D0J3L
- C22: renamed from C1; value C-USC0402 -> 0.1μF
- C24: renamed from C56; value 0.1μF -> 47pF
- C25: renamed from C57; value 0.1μF -> 47pF
- C26: renamed from C58; value 0.1μF -> 47pF
- C27: renamed from C59; value 0.1μF -> 15pF
- C28: renamed from C60; value 0.1μF -> 15pF
- C29: renamed from C61; value 0.1μF -> 15pF
- C30: renamed from C2; value C-USC0402 -> 0.1μF
- C31: renamed from C21; value C-USC0402 -> 0.1μF
- C32: renamed from C22; value C-USC0402 -> 0.1μF
- C36: renamed from C7; value C-USC0402 -> 47nF
- C37: renamed from C66; value C_Feedthrough -> NFM18PC106D0J3L
- C38: renamed from C8; value C-USC0402 -> 47nF
- C39: renamed from C9; value C-USC0402 -> 47nF
- C40: renamed from C14; value C-USC0402 -> 0.1μF
- C41: renamed from C15; value C-USC0402 -> 0.1μF
- C42: renamed from C3; value C-USC0402 -> 47nF
- C43: renamed from C6; value C-USC0402 -> 1nF
- C44: renamed from C16; value C-USC0402 -> 0.1μF
- C45: renamed from C20; value C-USC0402 -> 0.1μF
- C46: renamed from C4; value C-USC0402 -> 47nF
- C47: renamed from C23; value C-USC0402 -> 0.1μF
- C48: renamed from C24; value C-USC0402 -> 0.1μF
- C49: renamed from C5; value C-USC0402 -> 47nF
- C50: renamed from C25; value C-USC0402 -> 0.1μF
- C51: renamed from C26; value C-USC0402 -> 0.1μF
- C52: renamed from C10; value C-USC0402 -> 15pF
- C53: renamed from C27; value C-USC0402 -> 0.1μF
- C54: renamed from C11; value C-USC0402 -> 15pF
- C55: renamed from C28; value C-USC0402 -> 0.1μF
- C56: renamed from C30; value C-USC0402 -> 0.1μF
- C57: renamed from C42; value C-USC0402 -> 0.1μF
- C58: renamed from C43; value C-USC0402 -> 0.1μF
- C59: renamed from C44; value C-USC0402 -> 0.1μF
- C60: renamed from C45; value C-USC0402 -> 0.1μF
- C61: renamed from C46; value C-USC0402 -> 0.1μF
- C62: renamed from C47; value C-USC0402 -> 0.1μF
- C63: renamed from C48; value C-USC0402 -> 0.1μF
- C64: renamed from C49; value C-USC0402 -> 0.1μF
- C65: renamed from C50; value C-USC0402 -> 0.1μF
- FB1, FB2, FB3: value 220Ω -> BLM15BD221SN1D; footprint shinobi:R0402_2745533 -> Inductor_SMD:L_0402_1005Metric
- J2: renamed from J5; value USB_C_Receptacle_USB2.0_16P -> 217179-0001
- Q1: value UMH3N -> PUMH13-QF
- R10: renamed from R17; value R_Small -> 75Ω
- R11: renamed from R18; value R_Small -> 75Ω
- R12: renamed from R2; value R_Small -> 150Ω
- R13: renamed from R10; value R_Small -> 3kΩ
- R14: renamed from R9; value R_Small -> 75Ω
- R15: renamed from R3; value R_Small -> 200Ω
- R16: renamed from R4; value R_Small -> 75Ω
- R17: renamed from R5; value R_Small -> 200Ω
- R18: renamed from R6; value R_Small -> 75Ω
- R19: renamed from R7; value R_Small -> 200Ω
- R20: renamed from R8; value R_Small -> 75Ω
- R21: renamed from R1; value R_Small -> 4.7kΩ
- R22: renamed from R11; value R_Small -> 1MΩ
- R3: renamed from R13; value 12k -> 316kΩ
- R4: renamed from R19; value 12k -> 100kΩ
- R5: renamed from R22; value 12k -> 150kΩ
- R6: renamed from R23; value 12k -> 100kΩ
- R7: renamed from R15; value 12k -> 33Ω
- R8: renamed from R14; value 12k -> 33Ω
- R9: renamed from R16; value R_Small -> 75Ω
- RN1: renamed from RN2; value R_Pack04 -> EXB-28V123JX
- RN2: renamed from RN3; value R_Pack04 -> EXB-28V123JX
- U1: renamed from IC2; value TPS62825DMQT -> TPS62825DMQR
- U2: renamed from IC1; value TPS62825DMQT -> TPS62825DMQR
- Y1: renamed from Y3; value 26MHz -> ECS-260-7-36B-CKY-TR
- Y2: value CRYSTAL2.5X2.0 -> ECS-250-10-36B2-CTN-TR
- Y3: renamed from Y1; value CRYSTAL2.5X2.0 -> 830108208409
- moved FB3 8.60 mm to (149.1, 87.6), turned to 180 degrees
- moved FB1 8.59 mm to (157.7, 87.6), turned to 180 degrees
- moved R22 1.60 mm to (166.1, 89.9)
- moved C52 1.37 mm to (163.6, 88.0)
- moved C54 1.37 mm to (168.1, 88.0)
- moved Y3 1.37 mm to (165.8, 88.0)
- moved C50 0.24 mm to (169.5, 90.0)
- turned FB2 to 180 degrees
- renumbered C37 to C1, C31 to C10, C55 to C11, C35 to C12, C32 to C13, C64 to C14, C34 to C15, C13 to C16, C33 to C17, C65 to C2, C51 to C21, C53 to C23, C36 to C3, C18 to C33, C19 to C34, C40 to C35, C52 to C4, C12 to C5, C38 to C6, C39 to C7, C41 to C8, C54 to C9, J4 to J1, R20 to R1, R21 to R2, U6 to U3, U7 to U4, IC3 to U5, U5 to U6, U1 to U7, U2 to U8
Connections:
- C43 pad 2: /S -> S
- C52 pad 2: Net-(U1-XTOUT) -> Net-(U7-XTOUT)
- C54 pad 2: Net-(U1-XTIN) -> Net-(U7-XTIN)
- FB1 pad 1: ROUT -> B_VGA
- FB1 pad 2: R_VGA -> BOUT
- FB2 pad 1: GOUT -> G_VGA
- FB2 pad 2: G_VGA -> GOUT
- FB3 pad 1: BOUT -> R_VGA
- FB3 pad 2: B_VGA -> ROUT
- R14 pad 2: /S -> S
- R15 pad 1: /R -> R
- R16 pad 2: /R -> R
- R17 pad 1: /G -> G
- R18 pad 2: /G -> G
- R19 pad 1: /B -> B
- R20 pad 2: /B -> B
- R22 pad 1: unconnected-(R11-Pad1) -> Net-(U7-XTOUT)
- R22 pad 2: unconnected-(R11-Pad2) -> Net-(U7-XTIN)
- U7 pad 124: Net-(U1-XTIN) -> Net-(U7-XTIN)
- U7 pad 125: Net-(U1-XTOUT) -> Net-(U7-XTOUT)
- Y3 pad 1: Net-(U1-XTOUT) -> Net-(U7-XTOUT)
- Y3 pad 3: Net-(U1-XTIN) -> Net-(U7-XTIN)
Routing:
- net Net-(U1-XTIN): track 9.47 -> 0.00 mm
- net Net-(U1-XTOUT): track 7.98 -> 0.00 mm
- net Net-(U7-XTIN): track 0.00 -> 7.95 mm
- net Net-(U7-XTOUT): track 0.00 -> 6.59 mm
- net +2V5_FILT: track 16.0 -> 19.1 mm, vias 8 -> 9
- net +2V5: track 97.4 -> 99.6 mm
- net GND: vias 169 -> 216
Other:
- board text added: "1"
- board text added: "2"
- board text added: "2024"
- board text added: "3"
- board text added: "4"
- board text added: "GND"
- board text added: "Shinobi"
- board text added: "V+"
- board text added: "mks"
- board text added: "scaler"

Commit message: wip
Parts:
- C16, C17: value 10pF -> 15pF
- C6, C7: value 120pF -> 130pF
- Y1: value ECS-260-7-36B-CKY-TR -> 26MHz 10pF 2520
- Y2: value ECS-250-10-36B2-CTN-TR -> 25MHz 10pF 2520
- Y3: value 830108208409 -> 27MHz 10pF 2520
Routing:
- net VBUS: track 14.4 -> 28.0 mm
- net +2V5: track 99.6 -> 105.6 mm
- net +2V5_FILT: track 19.1 -> 21.2 mm
- net GND: vias 216 -> 225
Other:
- copper layers 4 -> 13
