File: KiCAD/shinobi.kicad_pcb (KiCad board)
At the start: 4 copper layers, 49.9 x 47 mm, 111 parts, among them J1 61300211121, J2 217179-0001, J3 61301011121, J4 61300711121, Q1 PUMH13-QF, U1 TPS62825DMQR, U2 TPS62825DMQR, U3 CH343P, U4 ESP8285, U5 74LVC2G17GW-Q100H, U6 SI5351A, U7 TV5725, U8 W9864G2JH-6, Y1 26MHz 10pF 2520, Y2 25MHz 10pF 2520, Y3 27MHz 10pF 2520

Commit message: small updates
Parts:
- added C66: 100uF, Capacitor_Tantalum_SMD:CP_EIA-2012-12_Kemet-R, F.Cu at (139.6, 113.1)
- added D1: LED, LED_SMD:LED_0603_1608Metric, F.Cu at (130.2, 123.2)
- added R23: 1kΩ, Resistor_SMD:R_0402_1005Metric, F.Cu at (127.8, 123.2)
- added SW1: SW_Push, Button_Switch_SMD:SW_SPST_B3U-1000P, F.Cu at (127.6, 95.3)
- C13: value 10μF -> 100uF; footprint Capacitor_SMD:C_0603_1608Metric -> Capacitor_Tantalum_SMD:CP_EIA-2012-12_Kemet-R
- moved R1 11.1 mm to (135.2, 104.2), turned to 0 degrees
- moved R2 2.97 mm to (131.1, 97.5), turned to 0 degrees
- moved C13 1.20 mm to (134.6, 115.0)
- moved C10 1.15 mm to (134.6, 113.8)
Connections:
- U4 pad 5: +2V5 -> unconnected-(U4-VDD_RTC-Pad5)
- U4 pad 9: unconnected-(U4-GPIO14-Pad9) -> Net-(U4-GPIO14)
Routing:
- net Net-(U4-GPIO14): track 0.00 -> 9.68 mm, vias 0 -> 2
- net Net-(J2-CC2): track 11.4 -> 2.52 mm
- net VBUS: track 26.5 -> 35.3 mm, vias 16 -> 17
- net Net-(J2-CC1): track 7.80 -> 6.22 mm
- net Net-(D1-A): track 0.00 -> 1.14 mm
- net RST: track 18.1 -> 18.6 mm
- net GND: vias 226 -> 233
Other:
- outline, holes or cut-outs redrawn
- board text added: "SW"
- board text added: "bitbuilt.net"

Commit message: updating files
Parts:
- D1: value LED -> green
- SW1: value SW_Push -> B3U-1000P
- renumbered C14 to C13, C13 to C14, C66 to C20, C20 to C22, C22 to C23, C23 to C24, C24 to C25, C25 to C26, C26 to C27, C27 to C28, C28 to C29, C29 to C30, C30 to C31, C31 to C32, C32 to C33, C33 to C34, C34 to C35, C35 to C36, C36 to C37, C37 to C38, C38 to C39, C39 to C40, C40 to C41, C41 to C42, C42 to C43, C43 to C44, C44 to C45, C45 to C46, C46 to C47, C47 to C48, C48 to C49, C49 to C50, C50 to C51, C51 to C52, C52 to C53, C53 to C54, C54 to C55, C55 to C56, C56 to C57, C57 to C58, C58 to C59, C59 to C60, C60 to C61, C61 to C62, C62 to C63, C63 to C64, C64 to C65, C65 to C66, R23 to R1, R9 to R10, R10 to R11, R11 to R12, R12 to R13, R13 to R14, R14 to R15, R15 to R16, R16 to R17, R17 to R18, R18 to R19, R1 to R2, R19 to R20, R20 to R21, R21 to R22, R22 to R23, R2 to R3, R3 to R4, R4 to R5, R5 to R6, R6 to R7, R7 to R8, R8 to R9
